Commit message: Progress report testing: save current progress

File: src/hospobot/src/rover_description/urdf/rover.urdf.xacro (robot description, xacro)
@@ -49,5 +49,22 @@
     <xacro:caster prefix="front" x_reflect="1" />
     <xacro:caster prefix="back" x_reflect="-1" />
-    <link name="laser_frame"/>
+    <link name="laser_frame">
+        <!-- A1M8 Scanner -->
+        <visual>
+            <origin xyz="0 0 -0.02" rpy="0 0 0"/>
+            <geometry>
+                <cylinder radius="0.035" length="0.04"/>
+            </geometry>
+            <material name="black"/>
+        </visual>
+        <!-- A1M8 Base & Motor -->
+        <visual>
+            <origin xyz="-0.025 0 -0.05" rpy="0 0 0"/>
+            <geometry>
+                <box size="0.10 0.06 0.02"/>
+            </geometry>
+            <material name="grey"/>
+        </visual>
+    </link>
     <joint name="laser_joint" type="fixed">
         <parent link="base_link"/>

Commit message: Add semantic perception pipeline and update web dashboard

File: src/hospobot/src/rover_description/urdf/rover.urdf.xacro (robot description, xacro)
@@ -73,3 +73,9 @@
         <origin xyz="0 0 0" rpy="0 0 0"/>
     </joint>
+    <link name="oakd_frame"/>
+    <joint name="oakd_joint" type="fixed">
+        <parent link="base_link"/>
+        <child link="oakd_frame"/>
+        <origin xyz="0 0 0.280" rpy="0 0.2618 0"/>
+    </joint>
 </robot>
