Commit message: Fix rotational odometry via Laser ICP, tune SLAM Toolbox, and add RViz FOV visualizer
- Switched to SLAM Toolbox online async mapping with Ceres solver
- Enabled Laser ICP Odometry (rtabmap_odom) to broadcast odom -> base_footprint TF directly from 2D LiDAR scans, eliminating diamond-drive wheel slip during turns
- Disabled wheel TF broadcasting in odrive_can_node and remapped telemetry to /odom_can
- Widened Ceres scan-matching coarse search angle to 45 deg and tuned angle penalty in mapper_params_online_async.yaml
- Added robot_fov_indicator_node to hospobot_perception to publish RViz MarkerArray of robot pose circle and three 2D LIDAR FOV cones (Front, Left, Right)
- Added .cache/ and *.db exclusions to .gitignore

File: src/hospobot/hospobot_urdf.xacro (robot description, xacro)
@@ -6,5 +6,5 @@
     <xacro:property name="shell_h" value="0.368"/>
     <xacro:property name="wheel_radius" value="0.0625"/>
-    <xacro:property name="track_width" value="0.280"/>
+    <xacro:property name="track_width" value="0.300"/>
     <xacro:property name="axle_z_offset" value="-0.0526"/>
     <link name="base_footprint"/>

File: src/hospobot/src/hospobot_description/urdf/hospobot.urdf.xacro (robot description, xacro)
@@ -6,11 +6,31 @@
     <xacro:property name="shell_h" value="0.368"/>
     <xacro:property name="wheel_radius" value="0.0625"/>
-    <xacro:property name="track_width" value="0.0826"/>
+    <xacro:property name="track_width" value="0.300"/>
     <xacro:property name="axle_z_offset" value="-0.0526"/>
+    <xacro:macro name="box_inertia" params="m w h d">
+      <inertial>
+        <origin xyz="0 0 0" rpy="0 0 0"/>
+        <mass value="${m}"/>
+        <inertia ixx="${(m/12) * (h*h + d*d)}" ixy="0.0" ixz="0.0" iyy="${(m/12) * (w*w + d*d)}" iyz="0.0" izz="${(m/12) * (w*w + h*h)}"/>
+      </inertial>
+    </xacro:macro>
+    <xacro:macro name="cylinder_inertia" params="m r h">
+      <inertial>
+        <origin xyz="0 0 0" rpy="${pi/2} 0 0" />
+        <mass value="${m}"/>
+        <inertia ixx="${(m/12) * (3*r*r + h*h)}" ixy="0" ixz="0" iyy="${(m/12) * (3*r*r + h*h)}" iyz="0" izz="${(m/2) * (r*r)}"/>
+      </inertial>
+    </xacro:macro>
+    <xacro:macro name="sphere_inertia" params="m r">
+      <inertial>
+        <mass value="${m}"/>
+        <inertia ixx="${(2/5) * m * (r*r)}" ixy="0.0" ixz="0.0" iyy="${(2/5) * m * (r*r)}" iyz="0.0" izz="${(2/5) * m * (r*r)}"/>
+      </inertial>
+    </xacro:macro>
     <link name="base_footprint"/>
     <joint name="base_joint" type="fixed">
         <parent link="base_footprint"/>
         <child link="base_link"/>
-        <origin xyz="0 0 ${ref_height}" rpy="0 0 0"/>
+        <origin xyz="0 0 ${ref_height - 0.10}" rpy="0 0 0"/>
     </joint>
     <link name="virtual_laser_link"/>
@@ -20,5 +40,16 @@
         <origin xyz="0 0 0.001" rpy="0 0 0"/>
     </joint>
-    <link name="base_link"/>
+    <link name="base_link">
+        <xacro:box_inertia m="10.0" w="${shell_w}" h="${shell_l}" d="${shell_h}"/>
+        <visual>
+            <origin xyz="0 0 ${shell_h/2 - 0.25}" rpy="0 0 ${pi/2}"/>
+            <geometry><mesh filename="package://hospobot_description/meshes/HospoBot_Full_Model.stl"/></geometry>
+            <material name="light_blue"><color rgba="0.6 0.8 1.0 1"/></material>
+        </visual>
+        <collision>
+            <origin xyz="0 0 ${shell_h/2}" rpy="0 0 0"/>
+            <geometry><box size="${shell_l} ${shell_w} ${shell_h}"/></geometry>
+        </collision>
+    </link>
     <xacro:macro name="wheel" params="prefix y_reflect">
         <link name="${prefix}_wheel">
@@ -30,4 +61,11 @@
                 <material name="black"><color rgba="0.1 0.1 0.1 1"/></material>
             </visual>
+            <collision>
+                <origin xyz="0 0 0" rpy="${pi/2} 0 0"/>
+                <geometry>
+                    <cylinder radius="${wheel_radius}" length="0.0172"/>
+                </geometry>
+            </collision>
+            <xacro:cylinder_inertia m="1.0" r="${wheel_radius}" h="0.0172"/>
         </link>
         <joint name="${prefix}_wheel_joint" type="continuous">
@@ -46,4 +84,8 @@
                 <material name="grey"><color rgba="0.5 0.5 0.5 1"/></material>
             </visual>
+            <collision>
+                <geometry><sphere radius="0.025"/></geometry>
+            </collision>
+            <xacro:sphere_inertia m="0.5" r="0.025"/>
         </link>
         <joint name="${prefix}_caster_joint" type="fixed">
@@ -67,16 +109,4 @@
         <origin xyz="0 0 -0.090" rpy="0 0 0"/>
     </joint>
-    <link name="chassis_visual">
-        <visual>
-            <origin xyz="0 0 ${shell_h/2}" rpy="0 0 0"/>
-            <geometry><box size="${shell_l} ${shell_w} ${shell_h}"/></geometry>
-            <material name="white"><color rgba="1 1 1 1"/></material>
-        </visual>
-    </link>
-    <joint name="chassis_joint" type="fixed">
-        <parent link="base_link"/>
-        <child link="chassis_visual"/>
-        <origin xyz="0 0 0" rpy="0 0 0"/>
-    </joint>
     <link name="oakd_frame"/>
     <joint name="oakd_joint" type="fixed">

Commit message: Fix YAML parsing error in velocity_smoother max_velocity and revert oakd voxel params

File: src/hospobot/hospobot_urdf.xacro (robot description, xacro)
@@ -53,5 +53,5 @@
         <parent link="base_link"/>
         <child link="laser_frame"/>
-        <origin xyz="0 0 0.300" rpy="0 0 0"/>
+        <origin xyz="0 0 0.300" rpy="0 0 3.14159265"/>
     </joint>
     <link name="imu_link"/>

File: src/hospobot/src/hospobot_description/urdf/hospobot.urdf.xacro (robot description, xacro)
@@ -101,5 +101,5 @@
         <parent link="base_link"/>
         <child link="laser_frame"/>
-        <origin xyz="0 0 0.500" rpy="0 0 0"/>
+        <origin xyz="0 0 0.500" rpy="0 0 3.14159265"/>
     </joint>
     <link name="imu_link"/>
